File: hardware/master-pcb/master-pcb.kicad_sch (KiCad schematic)
At the start: 19 parts, among them J1 RS-485 OUT, J2 INT IN 0-8, J4 UNDERGLOW OUT, SW1 PLAYER_ID, U1 Teensy 4.0, U2 THVD1429, U3 SN74AHCT125

Commit message: Master PCB: DigiKey BOM, SMA TVS, terminal footprints, DRC-clean layout
First commit of the routed master-pcb.kicad_pcb plus supporting library.

- Stackup + planes: JLC JLC04161H-7628; both inner layers -> GND
  (Sig+Pwr / GND / GND / Sig+Pwr); +3.3V distributes on outer copper.
- INT ESD: 3x SRV05-4 arrays -> 9 discrete unidirectional TVS D2-D10
  (Littelfuse SMAJ5.0A, DO-214AC / D_SMA_Handsoldering). Single-line shunt
  stubs at J2; closes the array-decoupling question.
- Terminal blocks built from datasheets: J2 -> Molex 39531 9-pos pluggable
  euro header (SD-39531-003, hole 1.60mm); J4 -> Adam Tech MRR52-5.08-2P
  (hole 1.50mm). Both replace stand-in footprints.
- BOM: MPN + DigiKey P/N fields on all 27 placed parts; stale panel-derived
  LCSC C-numbers cleared (master is DigiKey-sourced / hand-assembled).
  R4/R5 remain DNP. master-pcb-BOM.csv added.
- Layout: full route, GND stitching, mounting holes added.
- DRC (geometric + schematic-parity) 0/0/0, ERC 0.

Co-Authored-By: Claude Opus 4.8 <noreply@anthropic.com>
Parts:
- removed D2, D3, D4: SRV05-4, symbol Power_Protection:SRV05-4
- added D10, D2, D3, D4, D5, D6, D7, D8, D9: TVS 5V, Diode_SMD:D_SMA_Handsoldering, symbol Device:D_Zener
- added H1, H2, H3, H4: MountingHole, MountingHole:MountingHole_3.2mm_M3, symbol Mechanical:MountingHole
- added TP1: RS-485 A, TestPoint:TestPoint_THTPad_D2.0mm_Drill1.0mm, symbol Connector:TestPoint
- added TP2: RS-485 B, TestPoint:TestPoint_THTPad_D2.0mm_Drill1.0mm, symbol Connector:TestPoint
- added TP3: RS-485 DE, TestPoint:TestPoint_THTPad_D2.0mm_Drill1.0mm, symbol Connector:TestPoint
- added TP4: +3.3VDC, TestPoint:TestPoint_THTPad_D2.0mm_Drill1.0mm, symbol Connector:TestPoint
- added TP5: +5VDC_USB, TestPoint:TestPoint_THTPad_D2.0mm_Drill1.0mm, symbol Connector:TestPoint
- added TP6: GND, TestPoint:TestPoint_THTPad_D2.0mm_Drill1.0mm, symbol Connector:TestPoint
- added TP7: Underglow DATA 3.3V, TestPoint:TestPoint_THTPad_D2.0mm_Drill1.0mm, symbol Connector:TestPoint
- added TP8: Underglow DATA 5V, TestPoint:TestPoint_THTPad_D2.0mm_Drill1.0mm, symbol Connector:TestPoint
- C1, C2: footprint (none) -> Capacitor_SMD:C_0805_2012Metric; DigiKey (none) -> 399-C0805F104K1RACAUTOCT-ND; LCSC C14663 -> (none); MPN (none) -> C0805F104K1RACAUTO
- D1: footprint (none) -> LED_SMD:LED_0805_2012Metric; DigiKey (none) -> 732-4982-1-ND; MPN (none) -> 150080BS75000
- J1: footprint (none) -> Connector_Molex:Molex_Micro-Fit_3.0_43650-0300_1x03_P3.00mm_Horizontal; DigiKey (none) -> WM1861-ND; MPN (none) -> 0436500300
- J2: footprint (none) -> master-pcb:TerminalBlock_Molex_39531_1x09_P5.08mm_Vertical; DigiKey (none) -> WM25993-ND; MPN (none) -> 0395316009
- J4: footprint (none) -> master-pcb:TerminalBlock_MRR52-5.08-2P; DigiKey (none) -> 5245-MRR522-5.08-V-ND; MPN (none) -> MRR522-5.08-V
- R1: footprint (none) -> Resistor_SMD:R_0805_2012Metric; DigiKey (none) -> 311-120CRCT-ND; LCSC C22787 -> (none); MPN (none) -> RC0805FR-07120RL
- R2: footprint (none) -> Resistor_SMD:R_0805_2012Metric; DigiKey (none) -> 541-1.00KCCT-ND; LCSC C2907002 -> (none); MPN (none) -> CRCW08051K00FKEA
- R3: footprint (none) -> Resistor_SMD:R_0805_2012Metric; DigiKey (none) -> 311-330CRCT-ND; LCSC C23138 -> (none); MPN (none) -> RC0805FR-07330RL
- R4, R5: footprint Resistor_SMD:R_0603_1608Metric -> Resistor_SMD:R_0805_2012Metric
- RN1: footprint (none) -> Resistor_THT:R_Array_SIP10; DigiKey (none) -> 4610M-101-103LF-ND; MPN (none) -> 4610M-101-103LF
- SW1: footprint (none) -> Button_Switch_THT:SW_DIP_SPSTx03_Slide_9.78x9.8mm_W7.62mm_P2.54mm; DigiKey (none) -> 2223-DS01C-254-S-03BE-ND; MPN (none) -> DS01C-254-S-03BE
- U1: footprint (none) -> master-pcb:Teensy40_Socketed; symbol master-pcb:Teensy_4.0 -> master-pcb:Teensy4.0; DigiKey (none) -> 1568-15583-ND; MPN (none) -> 15583
- U2: footprint (none) -> Package_SO:SOIC-8_3.9x4.9mm_P1.27mm; DigiKey (none) -> 296-THVD1429DRCT-ND; LCSC C1850236 -> (none)
- U3: footprint (none) -> Package_DIP:DIP-14_W7.62mm; DigiKey (none) -> 296-4655-5-ND; LCSC C155176 -> (none); MPN (none) -> SN74AHCT125N
Connections:
- net +3.3VDC: now also U1.31 (VDD), TP4.1; no longer U1.26 (3V3)
- net +5VDC_USB: now also U1.33 (VIN), TP5.1; no longer U1.28 (VIN(USB5V))
- net GND: now also U1.32 (GND), D10.2 (A), D2.2 (A), D3.2 (A), D4.2 (A), D5.2 (A), D6.2 (A), D7.2 (A), D8.2 (A), D9.2 (A), TP6.1; no longer U1.27 (GND)
- net RS485+: now also TP1.1
- net RS485-: now also TP2.1
- net at R3.1, U3.3: now also TP8.1
- net GPIO 0/RX1: no longer names the net of U1.2 (GPIO_0)
- net GPIO 0/RX1: no longer U2.1 (RO)
- removed net GPIO 10: J2.8 (Pin_8), RN1.9 (R8), U1.12 (10)
- removed net GPIO 11: J2.9 (Pin_9), RN1.10 (R9), U1.13 (11)
- net GPIO 12: no longer names the net of U1.14 (GPIO_12)
- net GPIO 12: no longer U3.2
- removed net GPIO 13/LED: U1.15 (13/LED)
- net GPIO 14 renamed DIP_ID0
- net DIP_ID0: now also U1.8 (GPIO_6); no longer U1.16 (14)
- net GPIO 15 renamed DIP_ID1
- net DIP_ID1: now also U1.7 (GPIO_5); no longer U1.17 (15)
- net GPIO 16 renamed DIP_ID2
- net DIP_ID2: now also U1.6 (GPIO_4); no longer U1.18 (16)
- net GPIO 17 renamed STATUS_LED
- net STATUS_LED: now also U1.3 (GPIO_1); no longer U1.19 (17)
- net GPIO 18: no longer names the net of U1.20 (GPIO_13)
- net GPIO 19: no longer names the net of U1.21 (GPIO_14)
- net GPIO 1/TX1 renamed RS485_TX
- net RS485_TX: now also U1.10 (GPIO_8); no longer U1.3 (1/TX1)
- net GPIO 2 renamed RS485_DE
- net RS485_DE: now also U1.5 (GPIO_3), TP3.1; no longer U1.4 (2)
- net GPIO 20 renamed INT_DR
- net INT_DR: now also J2.1 (Pin_1), RN1.10 (R9), D2.1 (K)
- net GPIO 21 renamed INT_D
- net INT_D: now also J2.2 (Pin_2), RN1.9 (R8), D3.1 (K)
- net GPIO 22 renamed INT_DL
- net INT_DL: now also J2.3 (Pin_3), RN1.8 (R7), D4.1 (K)
- net GPIO 23 renamed INT_R
- net INT_R: now also J2.4 (Pin_4), RN1.7 (R6), D5.1 (K)
- removed net GPIO 3: J2.1 (Pin_1), RN1.2 (R1), U1.5 (3)
- removed net GPIO 4: J2.2 (Pin_2), RN1.3 (R2), U1.6 (4)
- removed net GPIO 5: J2.3 (Pin_3), RN1.4 (R3), U1.7 (5)
- removed net GPIO 6: J2.4 (Pin_4), RN1.5 (R4), U1.8 (6)
- net GPIO 7 renamed INT_C
- net INT_C: now also U1.26 (GPIO_19), D6.1 (K); no longer U1.9 (7)
- removed net GPIO 8: J2.6 (Pin_6), RN1.7 (R6), U1.10 (8)
- removed net GPIO 9: J2.7 (Pin_7), RN1.8 (R7), U1.11 (9)
- new net INT_L: D7.1 (K), J2.6 (Pin_6), RN1.5 (R4), U1.27 (GPIO_20)
- new net INT_U: D9.1 (K), J2.8 (Pin_8), RN1.3 (R2), U1.29 (GPIO_22)
- new net INT_UL: D10.1 (K), J2.9 (Pin_9), RN1.2 (R1), U1.30 (GPIO_23)
- new net INT_UR: D8.1 (K), J2.7 (Pin_7), RN1.4 (R3), U1.28 (GPIO_21)
- new net RS485_RX: U1.9 (GPIO_7), U2.1 (RO)
- new net UNDERGLOW_DATA: TP7.1, U1.13 (GPIO_11), U3.2
- no-connect marks 7 -> 11
Other:
- note added: "Microcontroller"
- note added: "Mounting"
- note added: "Overall Ground connection is added here to J4, as 2P terminal blocks are easy to find and source. We needed a way to connect the ground to the rest of the system anyway."
- note added: "Panel Interrupt Signals"
- note added: "RS-485 Receive & Transmit"
- note added: "RS-485 bias (R4/R5): fitted as DNP footprints, insurance only. THVD1429 has integrated open/short/idle failsafe, so the idle bus is already defined and no external bias is normally needed. Bias belongs at ONE point on the bus - the master is that point, so if the bench ever disagrees, populate here and nowhere else. 390R pair = approx. 236mV across the 60R terminated bus at 3.3V."
- note added: "Underglow LED Logic Shifter & Ground Hookup"
- moved on the sheet: C1, C2, D1, J1, J2, R1, R2, R3, R4, R5, RN1, SW1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
