File: hardware/master-pcb/master-pcb.kicad_sch (KiCad schematic)
At the start: 37 parts, among them J1 RS-485 OUT, J2 INT IN 0-8, J4 UNDERGLOW OUT, SW1 PLAYER_ID, U1 Teensy 4.0, U2 THVD1429, U3 SN74AHCT125

Commit message: Master: post-review rework — remove status LED, INT RC/TVS filter, pin reassign
- Remove status LED (D1, R2); Teensy onboard LED (pin 13) serves as status
- INT lines get two-stage protection: SMAJ5.0A TVS at the J2 entry + 330R
  series (R6-R14) + 1nF C0G RC (C3-C11) to GND on the Teensy-side node.
  Resolves review F3/F4 (series R makes the 5V-standoff TVS safe on the
  non-5V-tolerant Teensy pin; RC filters ESD/EMI). Pull-up stays Teensy-side.
- R15 10k pull-down on UNDERGLOW_DATA — defines U3 gate-A input LOW at boot
  (review F5)
- DIP -> GPIO 3/4/5, RS485_DE -> GPIO6; frees GPIO 0/1/2 and keeps Serial1
  (0/1) as the last spare hardware UART. RS-485 stays on Serial2 (7/8).
- ERC/DRC clean. docs/MASTER_PCB.md + BOM.md updated to match.
Parts:
- removed D1: STATUS, LED_SMD:LED_0805_2012Metric, symbol Device:LED
- removed R2: 1k, Resistor_SMD:R_0805_2012Metric, symbol Device:R
- added C10, C11, C3, C4, C5, C6, C7, C8, C9: 1nF C0G, Capacitor_SMD:C_0805_2012Metric, symbol Device:C
- added R10, R11, R12, R13, R14, R6, R7, R8, R9: 330R, Resistor_SMD:R_0805_2012Metric, symbol Device:R
- added R15: 10k, Resistor_SMD:R_0805_2012Metric, symbol Device:R
Connections:
- net DIP_ID0: now also U1.7 (GPIO_5); no longer U1.8 (GPIO_6)
- net DIP_ID1: now also U1.6 (GPIO_4); no longer U1.7 (GPIO_5)
- net DIP_ID2: now also U1.5 (GPIO_3); no longer U1.6 (GPIO_4)
- net GND: now also C10.2, C11.2, C3.2, C4.2, C5.2, C6.2, C7.2, C8.2, C9.2, R15.2
- net INT_C: now also C7.1, R10.2; no longer D6.1 (K), J2.5 (Pin_5)
- net INT_D: now also C4.1, R7.2; no longer D3.1 (K), J2.2 (Pin_2)
- net INT_DL: now also C5.1, R8.2; no longer D4.1 (K), J2.3 (Pin_3)
- net INT_DR: now also C3.1, R6.2; no longer D2.1 (K), J2.1 (Pin_1)
- net INT_L: now also C8.1, R11.2; no longer D7.1 (K), J2.6 (Pin_6)
- net INT_R: now also C6.1, R9.2; no longer D5.1 (K), J2.4 (Pin_4)
- net INT_U: now also C10.1, R13.2; no longer D9.1 (K), J2.8 (Pin_8)
- net INT_UL: now also C11.1, R14.2; no longer D10.1 (K), J2.9 (Pin_9)
- net INT_UR: now also C9.1, R12.2; no longer D8.1 (K), J2.7 (Pin_7)
- net RS485_DE: now also U1.8 (GPIO_6); no longer U1.5 (GPIO_3)
- net UNDERGLOW_DATA: now also R15.1
- net STATUS_LED: no longer names the net of U1.3 (GPIO_1)
- new net: D4.1 (K), J2.3 (Pin_3), R8.1
- new net: D2.1 (K), J2.1 (Pin_1), R6.1
- new net: D3.1 (K), J2.2 (Pin_2), R7.1
- new net: D10.1 (K), J2.9 (Pin_9), R14.1
- new net: D8.1 (K), J2.7 (Pin_7), R12.1
- new net: D5.1 (K), J2.4 (Pin_4), R9.1
- new net: D6.1 (K), J2.5 (Pin_5), R10.1
- new net: D7.1 (K), J2.6 (Pin_6), R11.1
- new net: D9.1 (K), J2.8 (Pin_8), R13.1
- no-connect marks 11 -> 12
Other:
- note added: "Unused"
- moved on the sheet: C2, D10, D2, D3, D4, D5, D6, D7, D8, D9, H1, H2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

Commit message: Master: RS-485 pair length-matched, RX/TX test points added
Same stackup as the panel (JLC04161H-7628), so the same 120-ohm target
geometry applies. The pair was already at W=0.15/S=0.2 -- it landed on the
right answer via the 0.15mm data-trace convention rather than by calculation
-- so only the skew needed work.

- /RS485+ and /RS485- now 45.39mm each: 0.000mm skew (was 0.60mm). F.Cu only,
  zero vias, ~119 ohm. Netclass diff-pair width corrected 0.2787 -> 0.15 and
  the stale USB pair class dropped (the Teensy handles USB internally; nothing
  USB is routed on this board).
- TP9 (RS485_RX) and TP10 (RS485_TX) added, giving probe access to the full
  transceiver interface alongside TP1/TP2/TP3 (A/B/DE).
- ~69% of the run is coupled at 0.2mm; the rest fans out to reach pads that
  are farther apart than the pair pitch (U2 pins 6/7, J1 Micro-Fit, R1,
  TP1/TP2). That is unavoidable and inconsequential at 1 Mbps -- documented as
  do-not-fix so it is not "corrected" later.

Also recorded: both inner layers are GND (GND_1/GND_2), unlike the panel's
GND/power split, so there is no reference-plane-type change anywhere on this
board.

Verified with all three ignored severities lifted, --severity-all
--schematic-parity --refill-zones: 0 violations, 0 unconnected, ERC 0. Only 3
cosmetic footprint_filters_mismatch notes (Euroblock, MRR52, DIP-3).
Parts:
- added TP10: RS-485 TX, TestPoint:TestPoint_THTPad_D2.0mm_Drill1.0mm, symbol Connector:TestPoint
- added TP9: RS-485 RX, TestPoint:TestPoint_THTPad_D2.0mm_Drill1.0mm, symbol Connector:TestPoint
Connections:
- net RS485_RX: now also TP9.1
- net RS485_TX: now also TP10.1
Changed lines of the file:
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@@
 	(wire
 		(pts
+			(xy 59.69 165.1) (xy 59.69 167.64)
+		)
+		(stroke
+			(width 0)
+			(type default)
+		)
+	)
+	(wire
+		(pts
 			(xy 190.5 41.91) (xy 194.31 41.91)
 		)
@@
 	(wire
 		(pts
+			(xy 48.26 175.26) (xy 59.69 175.26)
+		)
+		(stroke
+			(width 0)
+			(type default)
+		)
+	)
+	(wire
+		(pts
 			(xy 189.23 41.91) (xy 190.5 41.91)
 		)
@@
 	(wire
 		(pts
+			(xy 59.69 175.26) (xy 59.69 177.8)
+		)
+		(stroke
+			(width 0)
+			(type default)
+		)
+	)
+	(wire
+		(pts
 			(xy 355.6 33.02) (xy 374.65 33.02)
 		)
@@
 	(wire
 		(pts
+			(xy 48.26 165.1) (xy 59.69 165.1)
+		)
+		(stroke
+			(width 0)
+			(type default)
+		)
+	)
+	(wire
+		(pts
 			(xy 346.71 91.44) (xy 346.71 104.14)
 		)
@@
 	)
 	(symbol
+		(lib_id "Connector:TestPoint")
+		(at 48.26 175.26 90)
+		(unit 1)
+		(body_style 1)
+		(exclude_from_sim no)
+		(in_bom yes)
+		(on_board yes)
+		(in_pos_files yes)
+		(dnp no)
+		(property "Reference" "TP10"
+			(at 42.926 177.038 0)
+			(show_name no)
+			(do_not_autoplace no)
+			(effects
+				(font
+					(size 1.27 1.27)
+				)
+				(justify left)
+			)
+		)
+		(property "Value" "RS-485 TX"
+			(at 48.26 172.72 0)
+			(hide yes)
+			(show_name no)
+			(do_not_autoplace no)
+			(effects
+				(font
+					(size 1.27 1.27)
+				)
+				(justify left)
+			)
+		)
+		(property "Footprint" "TestPoint:TestPoint_THTPad_D2.0mm_Drill1.0mm"
+			(at 48.26 175.26 0)
+			(hide yes)
+			(show_name no)
+			(do_not_autoplace no)
+			(effects
+				(font
+					(size 1.27 1.27)
+				)
+			)
+		)
+		(property "Datasheet" ""
+			(at 48.26 175.26 0)
+			(hide yes)
+			(show_name no)
+			(do_not_autoplace no)
+			(effects
+				(font
+					(size 1.27 1.27)
+				)
+			)
+		)
+		(property "Description" "PARKED UNWIRED - probe test point, connect to RS-485 DE"
+			(at 48.26 175.26 0)
+			(hide yes)
+			(show_name no)
+			(do_not_autoplace no)
+			(effects
+				(font
+					(size 1.27 1.27)
+				)
+			)
+		)
+		(pin "1"
+		)
+		(instances
+			(project "master-pcb"
+				(path "/b2c3d4e5-0000-4000-8000-000000000002"
+					(reference "TP10")
+					(unit 1)
+				)
+			)
+		)
+	)
+	(symbol
 		(lib_id "power:GND")
 		(at 73.66 90.17 0)
@@
 					(unit 1)
 				)
+			)
+		)
+	)
+	(symbol
+		(lib_id "Connector:TestPoint")
+		(at 48.26 165.1 90)
+		(unit 1)
+		(body_style 1)
+		(exclude_from_sim no)
+		(in_bom yes)
+		(on_board yes)
+		(in_pos_files yes)
+		(dnp no)
+		(property "Reference" "TP9"
+			(at 42.926 166.878 0)
+			(show_name no)
+			(do_not_autoplace no)
+			(effects
+				(font
+					(size 1.27 1.27)
+				)
+				(justify left)
+			)
+		)
+		(property "Value" "RS-485 RX"
+			(at 48.26 162.56 0)
+			(hide yes)
+			(show_name no)
+			(do_not_autoplace no)
+			(effects
+				(font
+					(size 1.27 1.27)
+				)
+				(justify left)
+			)
+		)
+		(property "Footprint" "TestPoint:TestPoint_THTPad_D2.0mm_Drill1.0mm"
+			(at 48.26 165.1 0)
+			(hide yes)
+			(show_name no)
+			(do_not_autoplace no)
+			(effects
+				(font
+					(size 1.27 1.27)
+				)
+			)
+		)
+		(property "Datasheet" ""
+			(at 48.26 165.1 0)
+			(hide yes)
+			(show_name no)
+			(do_not_autoplace no)
+			(effects
+				(font
+					(size 1.27 1.27)
+				)
+			)
+		)
+		(property "Description" "PARKED UNWIRED - probe test point, connect to RS-485 DE"
+			(at 48.26 165.1 0)
+			(hide yes)
+			(show_name no)
+			(do_not_autoplace no)
+			(effects
+				(font
+					(size 1.27 1.27)
+				)
+			)
+		)
+		(pin "1"
+		)
+		(instances
+			(project "master-pcb"
+				(path "/b2c3d4e5-0000-4000-8000-000000000002"
+					(reference "TP9")
+					(unit 1)
+				)

Commit message: Both boards: J9/J4 to the vendor WJ500V land pattern; WS2815 cap question closed
Terminal blocks now use the footprint published by the manufacturer of the part
we actually buy (KANGNEX WJ500V-5.08-2P, LCSC C8465), pulled via easyeda2kicad,
replacing the hand-built Adam Tech MRR52 pattern:
- new panel-pcb/master-pcb:TerminalBlock_WJ500V-5.08-2P (hole 1.30mm per the
  vendor recommendation vs our 1.50mm, pad 2.00mm, origin centred between pins)
  plus the vendor 3D model, which supersedes the Phoenix MKDS stand-in
- panel J9 and master J4 reassigned, re-placed and re-routed
- part metadata follows: MPN WJ500V-5.08-2P, LCSC C8465, datasheet to the LCSC
  page, stale DigiKey fields dropped

Pitch (5.08mm) and body envelope (10.16 x 10.16mm) came out of the vendor data
matching our drawing-derived numbers, so that part of the physical-verification
item is closed without parts in hand; pin-1 orientation still wants an eyeball
on arrival.

Checklist: WS2815 5V bench test waived (not worth buying parts; the substantive
check was the datasheet-variant confirm, and VIH 2.7V min is a spec guarantee).
Per-LED pin-1 caps C22-C49 CLOSED as correct — the original 2018 WS2815 doc and
WS2815B-V3 both give pin 1 as "IC POWER SUPPLY, Suspended or connected with a
filter capacitor to GROUND"; our V1 doc is the outlier calling it NC. Paper does
not prove V1 silicon brings that rail out, but a 100nF is no DC load, so the cap
is inert at worst. No per-LED VDD decoupling is wanted: the channels are
constant-current, and the vendor states no extra components are needed.

DRC 0 / schematic-parity 0 / ERC 0 on both boards, zero exclusions.
Parts:
- J4: footprint master-pcb:TerminalBlock_MRR52-5.08-2P -> master-pcb:TerminalBlock_WJ500V-5.08-2P; DigiKey 5245-MRR522-5.08-V-ND -> (none); LCSC (none) -> C8465; MPN MRR522-5.08-V -> WJ500V-5.08-2P
Changed lines of the file:
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@@
 			)
 		)
-		(property "Footprint" "master-pcb:TerminalBlock_MRR52-5.08-2P"
+		(property "Footprint" "master-pcb:TerminalBlock_WJ500V-5.08-2P"
 			(at 225.55 41.42 0)
 			(hide yes)
@@
 			)
 		)
-		(property "Datasheet" "https://dcomponents.com/uploads/375571_MRR52-5.08-V.pdf"
+		(property "Datasheet" "https://www.lcsc.com/product-detail/C8465.html"
 			(at 225.55 41.42 0)
 			(hide yes)
@@
 			)
 		)
-		(property "Description" "Adam Tech MRR522-5.08-V, 2P 5.08mm top-entry screw terminal: GND + LED-DATA-OUT (5V logic). UI-gated; no sense pin"
+		(property "Description" "KANGNEX WJ500V-5.08-2P (LCSC C8465), 2P 5.08mm top-entry screw terminal: GND + LED-DATA-OUT (5V logic). UI-gated; no sense pin"
 			(at 225.55 41.42 0)
 			(hide yes)
@@
 			)
 		)
-		(property "LCSC" ""
+		(property "LCSC" "C8465"
 			(at -135.89 -120.65 0)
 			(hide yes)
@@
 			)
 		)
-		(property "MPN" "MRR522-5.08-V"
+		(property "MPN" "WJ500V-5.08-2P"
 			(at -135.89 -120.65 0)
 			(hide yes)
 			(show_name no)
-			(do_not_autoplace no)
-			(effects
-				(font
-					(size 1.27 1.27)
-				)
-			)
-		)
-		(property "DigiKey" "5245-MRR522-5.08-V-ND"
-			(at -166.37 -143.51 0)
-			(hide yes)
-			(show_name no)

Commit message: Both boards + docs: LCSC part identity sweep after the sourcing pivot
Every orderable part now carries the LCSC number it will actually be bought
under, and the fields that named DigiKey-era parts are gone.

Schematics + PCBs (mirrored so schematic-parity stays 0):
- LCSC fields filled: panel J2/J3/J4/J5/J6/J7/J8/J10/J11/SW1; master C1-C11,
  D2-D10, J1, R1, R3, R6-R15, RN1, SW1, U2, U3 (all 5 units of the multi-unit
  U3 -- the first pass only caught unit 3)
- DigiKey fields dropped everywhere they were superseded
- MPN cleared on generic passives, per the policy call: a 100nF 0805 X7R is not
  a specific part, so Value + LCSC carry its identity. MPN is kept only for
  genuinely named devices, including SMAJ5.0A as an industry-standard number
- Three parts were plain WRONG, not just stale: master RN1 4610M -> 4610X
  (different Bourns series), master SW1 CUI DS01C-254-S-03BE -> DORABO
  DS-3P-BU, panel SW1 CUI DS01C-254-S-04BE -> Zhongdi DS-04. Panel J2 also
  moved maker, Wurth 61300311121 -> XFCN PZ254V-11-03P
- panel SW1's Datasheet pointed at C99418, a different DIP switch entirely;
  RN1/SW1 datasheets repointed at their LCSC pages

Deliberately left blank, verified rather than assumed: test points, mounting
holes, panel FSR1 (reference-only DNP), master R4/R5 (390R, DNP -- not
ordered), master U1 (Teensy, PJRC/DigiKey is the real source) and master J2
(Euroblock from AliExpress, DigiKey kept as the documented fallback).

Docs: fixed the live spec tables in BOM.md sections A/B/C/G, MASTER_PCB.md and
PANEL_PCB.md, which still described J1 as the GCT USB4085, SW3 as the E-Switch
EG2201A, J9/J4 as the Adam Tech MRR52 and the switches as the CUI parts. The
labelled-superseded DigiKey quote in BOM section F is left intact as the
historical record that justified the pivot. Checklist: J1, J9+J4 and SW3
footprint items closed with what was actually done; PANEL_PCB.md's note about
the deleted SW_SS-22F04 footprint replaced with the resolution history.

DRC 0 / schemati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
Parts:
- C1, C2: DigiKey 399-C0805F104K1RACAUTOCT-ND -> (none); LCSC (none) -> C83055; MPN C0805F104K1RACAUTO -> (none)
- C10, C11, C3, C4, C5, C6, C7, C8, C9: LCSC (none) -> C1791
- D10, D2, D3, D4, D5, D6, D7, D8, D9: DigiKey SMAJ5.0ALFCT-ND -> (none); LCSC (none) -> C113952
- J1: DigiKey WM1861-ND -> (none); LCSC (none) -> C503478
- R1: DigiKey 311-120CRCT-ND -> (none); LCSC (none) -> C844816; MPN RC0805FR-07120RL -> (none)
- R10, R11, R12, R13, R14, R6, R7, R8, R9: LCSC (none) -> C844839
- R15: LCSC (none) -> C192906
- R3: DigiKey 311-330CRCT-ND -> (none); LCSC (none) -> C844839; MPN RC0805FR-07330RL -> (none)
- RN1: DigiKey 4610M-101-103LF-ND -> (none); LCSC (none) -> C840655; MPN 4610M-101-103LF -> 4610X-101-103LF
- SW1: DigiKey 2223-DS01C-254-S-03BE-ND -> (none); LCSC (none) -> C46595747; MPN DS01C-254-S-03BE -> DS-3P-BU
- U2: DigiKey 296-THVD1429DRCT-ND -> (none); LCSC (none) -> C1850236
- U3: DigiKey 296-4655-5-ND -> (none); LCSC (none) -> C354152
