File: hardware/master-pcb/master-pcb.kicad_pcb (KiCad board)
At the start: 4 copper layers, 77.5 x 65.5 mm, 64 parts, among them J1 RS-485 OUT, J10 B2B-XH-A, J11 B2B-XH-A, J2 UNDERGLOW OUT, J3 B2B-XH-A, J4 B2B-XH-A, J5 B2B-XH-A, J6 B2B-XH-A, J7 B2B-XH-A, J8 B2B-XH-A, J9 B2B-XH-A, SW1 PLAYER_ID, U1 THVD1429, U2 Teensy 4.0, U3 SN74AHCT1G125

Commit message: rev1: order both boards, and freeze exactly what went to fab
Boards are at JLCPCB as of 2026-08-18. Everything after this commit is rev 2.

Four design changes made on order day, all verified before submitting:

- U306 RP2040 signal pads 0.20 -> 0.23 mm, matching Raspberry Pi's official
  land pattern, via a local footprint. Length/pitch/centres/EP unchanged.
  Needed a zone refill and scoping the QSPI pour rule to B.Type == 'Zone'
  (it had no B-side condition, so it was policing track-to-pad too).
- RS-485 transceiver THVD1429 -> THVD1450DR on BOTH boards. Identical SOIC-8
  pinout. Gives up on-die IEC 61000-4-5 surge, which TI scopes to lightning and
  power-grid transients; gains 18 kV vs 8 kV contact ESD, the threat this pad
  actually documents. Also -$52 and 84x the stock, retiring the BOM's tightest
  line (60 units).
- 10 nF ADC filter caps C57112 -> C723749. The old part was X7R while the
  schematic said C0G; these are the four FSR ADC inputs, where Class II's
  piezoelectric response would inject charge synchronously with a footstep.
  Found by auditing all 35 BOM lines against live LCSC pages.
- master-pcb: 297 vias 0.45 -> 0.60 mm (0.075 -> 0.150 mm annular), after
  running DFM on the master for the first time. A quote is not a DFM check.

Both boards re-verified after every change: dual-panel 0/19/90/0,
master 0/0/0/0.

Adds hardware/fab-archive/rev1-2026-08-18/ with the byte-exact artifacts that
were manufactured, plus SHA256SUMS and a .gitattributes that disables CRLF
normalisation so they stay byte-exact. hardware/**/production/ is gitignored,
so without this there would be no record in git of what was physically built.

Adds QUOTE-2026-08-18.md (the real qty-20 quote; the July one is now marked
superseded) and splits the JLC order notes into PCB and PCBA remark blocks,
each within the 500-character limit the order form imposes.
Parts:
- U1: value THVD1429 -> THVD1450
