File: hardware/panel-pcb/panel-pcb.kicad_sch (KiCad schematic)
At the start: 137 parts, among them J1 USB_C_Receptacle_USB2.0_16P, J10 RS-485 OUT, J11 12V_OUT, J2 SWD, J3 FSR North, J4 FSR East, J5 12V_IN, J6 FSR South, J7 FSR West, J8 RS-485 IN, J9 INT OUT, SW1 PANEL_ID, SW2 BOOTSEL, SW3 RS-485 Termination, U1 RP2040, U2 THVD1429, U3 W25Q32JV, U4 SN74AHCT125, U5 AMS1117-5.0, U6 AP7361C-33ER-13, U7 USBLC6-2SC6, U8 LM66200, X1 12MHz ABM8-272-T3

Commit message: Panel PCB: JLC stackup, MRR52 terminal footprint on J9
- Stackup: KiCad default 0.48/0.48/0.48 FR4 -> real JLC JLC04161H-7628
  (0.2104 prepreg / 1.065 core, Er 4.4/4.6, 0.5oz inner). Fab output
  unaffected; corrects impedance calc / 3D / board thickness.
- J9 (INT out): repoint KF301 hand-stand-in -> TerminalBlock_MRR52-5.08-2P,
  built from Adam Tech datasheet 375571 (hole 1.3 -> 1.50mm, body 10.00mm).
  MPN MRR522-5.08-V, DigiKey 5245-MRR522-5.08-V-ND; stale KF301/C474881
  LCSC+datasheet cleared.
- Remove orphaned TerminalBlock_KF301-1P footprint (unused since J9 -> 2P).
- DRC/ERC clean.

Co-Authored-By: Claude Opus 4.8 <noreply@anthropic.com>
Parts:
- J9: footprint panel-pcb:TerminalBlock_KF301-2P_P5.08mm -> panel-pcb:TerminalBlock_MRR52-5.08-2P; DigiKey (none) -> 5245-MRR522-5.08-V-ND; LCSC C474881 -> (none); MPN KF301-5.0-2P -> MRR522-5.08-V
Changed lines of the file:
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@@
 			)
 		)
-		(property "Footprint" "panel-pcb:TerminalBlock_KF301-2P_P5.08mm"
+		(property "Footprint" "panel-pcb:TerminalBlock_MRR52-5.08-2P"
 			(at 220.98 234.95 0)
 			(hide yes)
@@
 			)
 		)
-		(property "Datasheet" "https://www.lcsc.com/datasheet/C474881.pdf"
+		(property "Datasheet" "https://dcomponents.com/uploads/375571_MRR52-5.08-V.pdf"
 			(at 220.98 234.95 0)
 			(hide yes)
@@
 			)
 		)
-		(property "Description" "Generic connector, single row, 01x02, script generated (kicad-library-utils/schlib/autogen/connector/)"
+		(property "Description" "Adam Tech MRR522-5.08-V, 2P 5.08mm Eurostyle PCB screw terminal (INT out, single conductor used)"
 			(at 220.98 234.95 0)
 			(hide yes)
@@
 			)
 		)
-		(property "MPN" "KF301-5.0-2P"
+		(property "MPN" "MRR522-5.08-V"
 			(at 220.98 234.95 0)
 			(hide yes)
@@
 			)
 		)
-		(property "LCSC" "C474881"
+		(property "LCSC" ""
 			(at 220.98 234.95 0)
 			(hide yes)
 			(show_name no)
+			(do_not_autoplace no)
+			(effects
+				(font
+					(size 1.27 1.27)
+				)
+			)
+		)
+		(property "DigiKey" "5245-MRR522-5.08-V-ND"
+			(at 0 0 0)
+			(hide yes)
+			(show_name no)

Commit message: Panel PCB: complete THT DigiKey/MPN fields
Populate DigiKey PN on hand-solder THT parts from the 2026-07-22 cart:
J1 (USB-C), J2 (SWD, Würth 61300311121), J5/J11 + J8/J10 (Micro-Fit),
SW3 (EG2201A). SW1 corrected from stale DSWB04LHGET -> CUI DS01C-254-S-04BE
(the actual cart part) with DigiKey PN, stale LCSC C99418 cleared.
FSR JST (J3/J4/J6/J7) keep MPN only — out of stock at DigiKey, sourced
elsewhere. ERC clean.

Co-Authored-By: Claude Opus 4.8 <noreply@anthropic.com>
Parts:
- J1: DigiKey (none) -> 2073-USB4085-GF-ACT-ND
- J10, J8: DigiKey (none) -> WM1861-ND
- J11, J5: DigiKey (none) -> WM1860-ND
- J2: DigiKey (none) -> 732-5316-ND; MPN (none) -> 61300311121
- SW1: DigiKey (none) -> 2223-DS01C-254-S-04BE-ND; LCSC C99418 -> (none); MPN DSWB04LHGET -> DS01C-254-S-04BE
- SW3: DigiKey (none) -> EG1905-ND
Changed lines of the file:
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@@
 			)
 		)
+		(property "DigiKey" "WM1861-ND"
+			(at 0 0 0)
+			(hide yes)
+			(show_name no)
+			(do_not_autoplace no)
+			(effects
+				(font
+					(size 1.27 1.27)
+				)
+			)
+		)
 		(pin "1"
 		)
@@
 			)
 		)
+		(property "DigiKey" "WM1860-ND"
+			(at 0 0 0)
+			(hide yes)
+			(show_name no)
+			(do_not_autoplace no)
+			(effects
+				(font
+					(size 1.27 1.27)
+				)
+			)
+		)
 		(pin "1"
 		)
@@
 			)
 		)
+		(property "DigiKey" "2073-USB4085-GF-ACT-ND"
+			(at 0 0 0)
+			(hide yes)
+			(show_name no)
+			(do_not_autoplace no)
+			(effects
+				(font
+					(size 1.27 1.27)
+				)
+			)
+		)
 		(pin "A1"
 		)
@@
 			)
 		)
+		(property "DigiKey" "WM1861-ND"
+			(at 0 0 0)
+			(hide yes)
+			(show_name no)
+			(do_not_autoplace no)
+			(effects
+				(font
+					(size 1.27 1.27)
+				)
+			)
+		)
 		(pin "1"
 		)
@@
 			)
 		)
+		(property "DigiKey" "WM1860-ND"
+			(at 0 0 0)
+			(hide yes)
+			(show_name no)
+			(do_not_autoplace no)
+			(effects
+				(font
+					(size 1.27 1.27)
+				)
+			)
+		)
 		(pin "1"
 		)
@@
 			)
 		)
+		(property "DigiKey" "EG1905-ND"
+			(at 0 0 0)
+			(hide yes)
+			(show_name no)
+			(do_not_autoplace no)
+			(effects
+				(font
+					(size 1.27 1.27)
+				)
+			)
+		)
 		(pin "1"
 		)
@@
 			)
 		)
+		(property "MPN" "61300311121"
+			(at 0 0 0)
+			(hide yes)
+			(show_name no)
+			(do_not_autoplace no)
+			(effects
+				(font
+					(size 1.27 1.27)
+				)
+			)
+		)
+		(property "DigiKey" "732-5316-ND"
+			(at 0 0 0)
+			(hide yes)
+			(show_name no)
+			(do_not_autoplace no)
+			(effects
+				(font
+					(size 1.27 1.27)
+				)
+			)
+		)
 		(pin "1"
 		)
@@
 			)
 		)
-		(property "MPN" "DSWB04LHGET"
+		(property "MPN" "DS01C-254-S-04BE"
 			(at 38.1 33.02 0)
 			(hide yes)
@@
 			)
 		)
-		(property "LCSC" "C99418"
+		(property "LCSC" ""
 			(at 38.1 33.02 0)
 			(hide yes)
 			(show_name no)
+			(do_not_autoplace no)
+			(effects
+				(font
+					(size 1.27 1.27)
+				)
+			)
+		)
+		(property "DigiKey" "2223-DS01C-254-S-04BE-ND"
+			(at 0 0 0)
+			(hide yes)
+			(show_name no)
