File: hardware/dual-panel/carrier.kicad_sch (KiCad schematic)
At the start: 78 parts, among them J10 RS-485 OUT, J11 12V_OUT, J12 Conn_01x17, J13 Conn_01x17, J16 SWD, J3 FSR North, J4 FSR East, J5 12V_IN, J6 FSR South, J7 FSR West, J8 RS-485 IN, J9 INT OUT, SW1 PANEL_ID, SW3 RS-485 Termination

Commit message: dual-panel: brain laid out, interface reworked to 4x 1x8, carrier routed
Work in progress checkpoint — not clean yet, see below.

Interface replaced: the two 1x17 rows became four 1x8 connectors, placed
in the two continuous free bands across the carrier (y~49-58 and y~83-92).
Carrier headers J12/J13/J14/J15 mate with brain sockets J2/J19/J17/J18;
both boards use the same relative layout, since the brain is translated
under the carrier rather than flipped. Grouped by function so the FSR
lines and the fast signals land on separate connectors.

Brain outline drawn at 76.1 x 63.6mm with its own GND_Brain pour, sitting
inside the measured 88 x 100mm frame opening with ~6mm per side in X.
Two M3 holes added per board (carrier H5/H6, brain H1/H2), registered to
the connectors; screw enters from the brain underside with a nut above
the carrier.

Cavity measured: 6mm from the carrier underside to the frame floor, plus
14mm to the cavity bottom, so 20mm of depth inside the opening. That
retires the depth gate and also means the carrier's four remaining
bottom-side parts (D30, R17, R20, C57, tallest 2.3mm) can stay put.

Known open, to fix next:
- +3.3VDC may be split into three islands with the regulator in only one
- +12VDC and VBUS each broken on the brain; VBUS leaves U8 unfed
- FSR_West does not land on R8 pad 1; J1 shell pad floating
- QSPI_SCLK clears GND_Brain by 0 in four places
- 180-degree rotation is only blocked by 0.50mm at the connectors; wants
  a 2.54mm Y delta between J15 and J14 for a half-pitch refusal
- screw scheme needs a board-to-board spacer, and the nuts land inside
  the LED field
- silkscreen deliberately untouched (110 of 115 DRC violations)

ERC 0, schematic parity 0. 25 unconnected, of which roughly 19 are the
expected cross-gap airwires at the mating connectors.
Parts:
- removed J12, J13: Conn_01x17, Connector_PinHeader_2.54mm:PinHeader_1x17_P2.54mm_Vertical, symbol Connector_Generic:Conn_01x17
- added H1, H2: MountingHole_Pad, MountingHole:MountingHole_3.2mm_M3_Pad, symbol Mechanical:MountingHole_Pad
- added J12, J13, J14, J15: Conn_01x08_Pin, Connector_PinHeader_2.54mm:PinHeader_1x08_P2.54mm_Vertical, symbol Connector:Conn_01x08_Pin
Connections:
- net +12VDC: now also J14.1 (Pin_1), J15.6 (Pin_6)
- net +3.3VDC: now also J12.1 (Pin_1), J15.1 (Pin_1)
- net DEBUG_LED: now also J15.8 (Pin_8)
- net DIP_ID0: now also J13.4 (Pin_4)
- net DIP_ID1: now also J13.3 (Pin_3)
- net DIP_ID2: now also J13.2 (Pin_2)
- net DIP_ID3: now also J13.1 (Pin_1)
- net FSR_East: now also J12.8 (Pin_8)
- net FSR_North: now also J15.2 (Pin_2)
- net FSR_South: now also J13.8 (Pin_8)
- net FSR_West: now also J15.3 (Pin_3)
- net GND: now also H1.1, H2.1, J12.2 (Pin_2), J12.4 (Pin_4), J12.7 (Pin_7), J13.5 (Pin_5), J13.7 (Pin_7), J14.2 (Pin_2), J14.3 (Pin_3), J14.4 (Pin_4), J14.6 (Pin_6), J15.4 (Pin_4), J15.5 (Pin_5), J15.7 (Pin_7)
- net INT_OUT: now also J13.6 (Pin_6)
- net LED_DATA_5V: now also J14.5 (Pin_5)
- net RS485+: now also J12.5 (Pin_5)
- net RS485-: now also J12.6 (Pin_6)
- net SWCLK: now also J14.7 (Pin_7)
- net SWDIO: now also J14.8 (Pin_8)
- net TERM_SENSE: now also J12.3 (Pin_3)
- no-connect marks 13 -> 5

Commit message: dual-panel: carrier test points + brain labelling
Carrier test points, 5 -> 18. The brain is buried under the carrier, so its
test points need the stack apart; these are the ones reachable on a working pad.

- reachable-only-here: TP18/TP19 RS485+/-, TP20 +3.3VDC (the FSR excitation
  rail, which had no carrier test point at all), TP21 on the INT terminal side
  of R17
- LED chain bisect: TP22/TP23/TP24/TP25 on LD6, LD12, LD18, LD23, so a dead
  chain localises in a couple of probes instead of hunting 25 parts
- TP26 +12VDC at the far end of the spine, to measure real IR drop across the
  LED field against the ~18mV the comb topology was chosen on
- TP27 TERM_SENSE, and TP28/TP29/TP30 GND so each probe cluster has a local
  return

Deliberately left off: the four FSR lines (highest-impedance nets on the board,
dividers are on the brain so the carrier side is raw sensor line, and the
isolation from LED data was deliberate - probe the JST-PH connectors instead)
and DIP_ID0-3 (probe SW1 directly).

Also silkscreen labelling on the brain.

Verified: DRC 0, ERC 0, 19 unconnected and all cross-gap. Test points are
synced 30/30 between schematic and PCB with matching UUID links. Parity is 93,
up one only because TP21 joined Net-(D30-K), a net already in the pre-existing
cosmetic naming class.
Parts:
- added TP18, TP19, TP20, TP21, TP22, TP23, TP24, TP25, TP28, TP29, TP30: GND, TestPoint:TestPoint_THTPad_D2.0mm_Drill1.0mm, symbol Connector:TestPoint
- added TP26, TP27: +12VDC, TestPoint:TestPoint_THTPad_D2.0mm_Drill1.0mm, symbol Connector:TestPoint
Connections:
- net +12VDC: now also TP26.1
- net +3.3VDC: now also TP20.1
- net GND: now also TP28.1, TP29.1, TP30.1
- net LD12: now also TP23.1
- net LD18: now also TP24.1
- net LD23: now also TP25.1
- net LD6: now also TP22.1
- net RS485+: now also TP18.1
- net RS485-: now also TP19.1
- net TERM_SENSE: now also TP27.1
- net at D30.1 (K), J9.1 (Pin_1), R17.2: now also TP21.1
Other:
- note removed: "Offset J12/J13 from the brain centerline at layout, so a rotated board can't seat."
- moved on the sheet: TP15, TP16, TP17

Commit message: Fix R20 LCSC code, and let gen_fab.py export any board
R20 (1M, the RS-485 shield bleed) carried C4216, which is R19's 33k part - the
3302 marking confirms C4216 is genuinely 33k, so R19 was right and R20 had
inherited it. Now C22935. The bug was in BOTH designs, since dual-panel was
seeded from panel-pcb, so all four live files are fixed: carrier.kicad_sch,
dual-panel.kicad_pcb, panel-pcb.kicad_sch, panel-pcb.kicad_pcb. R19 keeps C4216
everywhere.

Left as-is, nine panels would each have shunted the cable shield to ground
through 33k instead of 1M - about 3.7k in parallel rather than 111k - largely
defeating the hybrid grounding the shield scheme was built around, with nothing
visibly wrong on the board.

gen_fab.py gains --board and --out so it can export panel-pcb for a comparison
quote using identical filtering, plus --allow-part-clash to downgrade the LCSC
collision check for comparison quotes only.

Verified after the edits: dual-panel DRC 0 / ERC 0 / 19 cross-gap unconnected,
panel-pcb DRC 0 / ERC 0 / parity 0 / unconnected 0. Both fab packages now export
with no collision and every BOM line carrying an LCSC number.
Parts:
- R20: LCSC C4216 -> C22935
Changed lines of the file:
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@@
 			)
 		)
-		(property "LCSC" "C4216"
+		(property "LCSC" "C22935"
 			(at 90.17 49.53 0)
 			(hide yes)

Commit message: dual-panel: per-sheet refdes blocks, stitching vias, silkscreen
Reference designators are now numbered in per-sheet blocks — carrier 2xx,
brain 3xx — so a designator says which of the two boards a part sits on.
That is the multi-sheet exception the review conventions allow, and it is
cheaper than closing every gap left by seeding both sheets from panel-pcb
and stripping them down. No designator is duplicated across the sheets.

Also: ground stitching vias (464 -> 1071), the year appended to both
name/rev blocks, and the fab order-number placeholder removed.

Note for the next renumber: "Update PCB from Schematic" will refuse to
match and offer to re-add every footprint. The links are fine — it is the
sticky "re-link by reference designator" option, which cannot match once
every designator has changed. Recovery is to revert the annotation,
re-link once while the designators still agree, then reannotate. The
underlying cause is that dual-panel.kicad_pro registers the root sheet as
a1b2c3d4-...-000000000001, which is panel-pcb's root UUID, while
dual-panel.kicad_sch says ...00000000d001.

DRC 0, ERC 0 with zones refilled. 19 unconnected and 93 net_conflict
remain, unchanged from before this commit: the 19 are the board-to-board
mating gap KiCad cannot model, the 93 are pre-existing net-name
disagreements on the WS2815 VCC/PWR_FLAG nets.
Parts:
- renumbered C51 to C201, C57 to C202, C22 to C203, C23 to C204, C24 to C205, C25 to C206, C26 to C207, C27 to C208, C28 to C209, C29 to C210, C30 to C211, C31 to C212, C32 to C213, C33 to C214, C34 to C215, C35 to C216, C36 to C217, C39 to C218, C40 to C219, C41 to C220, C42 to C221, C43 to C222, C45 to C223, C46 to C224, C47 to C225, C48 to C226, C49 to C227, D30 to D201, D1 to D202, D2 to D203, D3 to D204, D4 to D205, D5 to D206, D6 to D207, D7 to D208, D8 to D209, D9 to D210, D10 to D211, D11 to D212, D13 to D213, D14 to D214, D15 to D215, D16 to D216, D17 to D217, D18 to D218, D19 to D219, D20 to D220, D21 to D221, D22 to D222, D24 to D223, D25 to D224, D26 to D225, D27 to D226, D28 to D227, FSR2 to FSR201, H1 to H201, H2 to H202, J7 to J201, J6 to J202, J4 to J203, J8 to J204, J5 to J205, J3 to J206, J10 to J207, J11 to J208, J16 to J209, J12 to J210, J13 to J211, J14 to J212, J15 to J213, J9 to J214, R2 to R201, R20 to R202, R17 to R203, R15 to R204, SW1 to SW201, SW3 to SW202, TP27 to TP201, TP18 to TP202, TP26 to TP203, TP19 to TP204, TP8 to TP205, TP20 to TP206, TP28 to TP207, TP29 to TP208, TP30 to TP209, TP15 to TP210, TP21 to TP211, TP16 to TP212, TP17 to TP213, TP9 to TP214, TP22 to TP215, TP23 to TP216, TP24 to TP217, TP25 to TP218

Commit message: dual-panel: third mounting hole, fix hole refdes, set via fill/cap
Adds a third M3 fixing to both boards and moves the top one, which removes
the rocking degree of freedom the two-screw mount still had. With only two
screws the boards could rotate about the axis through them, and the two
board-to-board sockets furthest off that axis sat 27mm and 34mm out. Three
non-collinear fixings constrain the plane outright.

  arrangement                 worst socket-to-screw   support triangle
  2 screws (before)                   45.99 mm        none (collinear)
  old top + new bottom-right          41.46 mm        1576 mm2
  top moved + new bottom-right        32.07 mm        1583 mm2

Brain/carrier hole pairs stay on the exact (101.68, -16.87) offset.

Mounting hole refdes were swapped against the 2xx=carrier / 3xx=brain
convention: H201/H202 sat on the brain and H301/H302 on the carrier. The
schematic sheets were already right, so this swaps the footprint placements
only, leaving the symbol-to-footprint paths untouched. Their reference-text
offsets were swapped too, since those were tuned per location (a -0.81mm
nudge to clear J302's label, and one text placed below to stay off the
brain's top edge) and would otherwise have collided in their new homes.

Sets board-level via capping and filling ahead of ordering with JLC's epoxy
fill option. This is annotation only -- verified it changes nothing in the
Gerbers, drill, gerber job file, IPC-2581 or ODB++ output. Set at board level
rather than per-via because every via reads FROM_BOARD, and because the fill
is a whole-board process, not a per-via selection.

Also restores via tenting, which had been switched off. That opened a solder
mask window over all 1107 vias -- a bridging risk in assembly, and the cause
of 138 silkscreen-clipped-by-mask violations.

Stitching vias re-added after the clearance rework: 1107 total (1014 GND).
Carrier stitching matches the pre-rework board exactly (790 GND vias, median
GND-pad-to-via 1.55mm,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
Parts:
- added H203: MountingHole_Pad, MountingHole:MountingHole_3.2mm_M3_Pad, symbol Mechanical:MountingHole_Pad
Connections:
- net GND: now also H203.1
Other:
- moved on the sheet: H201, H202
Changed lines of the file:
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@@
 	)
 	(junction
-		(at 149.86 252.73)
-		(diameter 0)
-		(color 0 0 0 0)
-	)
-	(junction
 		(at 379.73 80.01)
 		(diameter 0)
@@
 	)
 	(junction
+		(at 146.05 256.54)
+		(diameter 0)
+		(color 0 0 0 0)
+	)
+	(junction
 		(at 326.39 87.63)
 		(diameter 0)
@@
 	(wire
 		(pts
-			(xy 135.89 250.19) (xy 135.89 252.73)
+			(xy 119.38 254) (xy 119.38 256.54)
 		)
 		(stroke
@@
 	(wire
 		(pts
+			(xy 171.45 254) (xy 171.45 256.54)
+		)
+		(stroke
+			(width 0)
+			(type default)
+		)
+	)
+	(wire
+		(pts
 			(xy 243.84 87.63) (xy 243.84 71.12)
 		)
@@
 	(wire
 		(pts
-			(xy 162.56 252.73) (xy 162.56 250.19)
+			(xy 146.05 256.54) (xy 146.05 254)
 		)
 		(stroke
@@
 	(wire
 		(pts
-			(xy 149.86 252.73) (xy 135.89 252.73)
+			(xy 146.05 256.54) (xy 119.38 256.54)
 		)
 		(stroke
@@
 	(wire
 		(pts
-			(xy 149.86 252.73) (xy 162.56 252.73)
-		)
-		(stroke
-			(width 0)
-			(type default)
-		)
-	)
-	(wire
-		(pts
 			(xy 127 77.47) (xy 127 72.39)
 		)
@@
 	(wire
 		(pts
+			(xy 171.45 256.54) (xy 146.05 256.54)
+		)
+		(stroke
+			(width 0)
+			(type default)
+		)
+	)
+	(wire
+		(pts
 			(xy 48.26 80.01) (xy 46.99 80.01)
 		)
@@
 	(symbol
 		(lib_id "Mechanical:MountingHole_Pad")
-		(at 135.89 247.65 0)
+		(at 119.38 251.46 0)
 		(unit 1)
 		(body_style 1)
@@
 		(fields_autoplaced yes)
 		(property "Reference" "H201"
-			(at 138.43 245.1099 0)
+			(at 121.92 248.9199 0)
 			(show_name no)
 			(do_not_autoplace no)
@@
 		)
 		(property "Value" "MountingHole_Pad"
-			(at 138.43 247.6499 0)
+			(at 121.92 251.4599 0)
 			(show_name no)
 			(do_not_autoplace no)
@@
 		)
 		(property "Footprint" "MountingHole:MountingHole_3.2mm_M3_Pad"
-			(at 135.89 247.65 0)
+			(at 119.38 251.46 0)
 			(hide yes)
 			(show_name no)
@@
 		)
 		(property "Datasheet" ""
-			(at 135.89 247.65 0)
+			(at 119.38 251.46 0)
 			(hide yes)
 			(show_name no)
@@
 		)
 		(property "Description" "Mounting Hole with connection"
-			(at 135.89 247.65 0)
+			(at 119.38 251.46 0)
 			(hide yes)
 			(show_name no)
@@
 	)
 	(symbol
+		(lib_id "Mechanical:MountingHole_Pad")
+		(at 171.45 251.46 0)
+		(unit 1)
+		(body_style 1)
+		(exclude_from_sim no)
+		(in_bom no)
+		(on_board yes)
+		(in_pos_files yes)
+		(dnp no)
+		(fields_autoplaced yes)
+		(property "Reference" "H203"
+			(at 173.99 248.9199 0)
+			(show_name no)
+			(do_not_autoplace no)
+			(effects
+				(font
+					(size 1.27 1.27)
+				)
+				(justify left)
+			)
+		)
+		(property "Value" "MountingHole_Pad"
+			(at 173.99 251.4599 0)
+			(show_name no)
+			(do_not_autoplace no)
+			(effects
+				(font
+					(size 1.27 1.27)
+				)
+				(justify left)
+			)
+		)
+		(property "Footprint" "MountingHole:MountingHole_3.2mm_M3_Pad"
+			(at 171.45 251.46 0)
+			(hide yes)
+			(show_name no)
+			(do_not_autoplace no)
+			(effects
+				(font
+					(size 1.27 1.27)
+				)
+			)
+		)
+		(property "Datasheet" ""
+			(at 171.45 251.46 0)
+			(hide yes)
+			(show_name no)
+			(do_not_autoplace no)
+			(effects
+				(font
+					(size 1.27 1.27)
+				)
+			)
+		)
+		(property "Description" "Mounting Hole with connection"
+			(at 171.45 251.46 0)
+			(hide yes)
+			(show_name no)
+			(do_not_autoplace no)
+			(effects
+				(font
+					(size 1.27 1.27)
+				)
+			)
+		)
+		(pin "1"
+		)
+		(instances
+			(project "dual-panel"
+				(path "/a1b2c3d4-0000-4000-8000-000000000001/a1b2c3d4-0000-4000-8000-00000000dc01"
+					(reference "H203")
+					(unit 1)
+				)
+			)
+		)
+	)
+	(symbol
 		(lib_id "power:+3V3")
 		(at 254 220.98 0)
@@
 	(symbol
 		(lib_id "Mechanical:MountingHole_Pad")
-		(at 162.56 247.65 0)
+		(at 146.05 251.46 0)
 		(unit 1)
 		(body_style 1)
@@
 		(fields_autoplaced yes)
 		(property "Reference" "H202"
-			(at 165.1 245.1099 0)
+			(at 148.59 248.9199 0)
 			(show_name no)
 			(do_not_autoplace no)
@@
 		)
 		(property "Value" "MountingHole_Pad"
-			(at 165.1 247.6499 0)
+			(at 148.59 251.4599 0)
 			(show_name no)
 			(do_not_autoplace no)
@@
 		)
 		(property "Footprint" "MountingHole:MountingHole_3.2mm_M3_Pad"
-			(at 162.56 247.65 0)
+			(at 146.05 251.46 0)
 			(hide yes)
 			(show_name no)
@@
 		)
 		(property "Datasheet" ""
-			(at 162.56 247.65 0)
+			(at 146.05 251.46 0)
 			(hide yes)
 			(show_name no)
@@
 		)
 		(property "Description" "Mounting Hole with connection"
-			(at 162.56 247.65 0)
+			(at 146.05 251.46 0)
 			(hide yes)
 			(show_name no)
@@
 	(symbol
 		(lib_id "power:GND")
-		(at 149.86 252.73 0)
+		(at 146.05 256.54 0)
 		(unit 1)
 		(body_style 1)
@@
 		(dnp no)
 		(property "Reference" "#PWR0216"
-			(at 149.86 257.81 0)
+			(at 146.05 261.62 0)
 			(hide yes)
 			(show_name no)
@@
 		)
 		(property "Value" "GND"
-			(at 149.86 256.54 0)
+			(at 146.05 260.35 0)
 			(show_name no)
 			(do_not_autoplace no)
@@
 		)
 		(property "Footprint" ""
-			(at 149.86 252.73 0)
+			(at 146.05 256.54 0)
 			(hide yes)
 			(show_name no)
@@
 		)
 		(property "Datasheet" ""
-			(at 149.86 252.73 0)
+			(at 146.05 256.54 0)
 			(hide yes)
 			(show_name no)
@@
 		)
 		(property "Description" "Power symbol creates a global label with name \"GND\" , ground"
-			(at 149.86 252.73 0)
+			(at 146.05 256.54 0)
 			(hide yes)
 			(show_name no)
